Commit message: camera meshes path fixed

File: rover_description/urdf/sensors/depth_camera.urdf.xacro (robot description, xacro)
@@ -13,5 +13,5 @@
         <origin rpy="${math_pi_over_2} 0 ${math_pi_over_2}" xyz="0 0 0"/>
         <geometry>
-          <mesh filename="package://rb1_torso_description/meshes/sensors/asus_xtion_pro_live.dae" scale="0.001 0.001 0.001"/>
+          <mesh filename="package://rover_description/meshes/sensors/camera/asus_xtion_pro_live.dae" scale="0.001 0.001 0.001"/>
         </geometry>
       </visual>
@@ -19,5 +19,5 @@
         <origin rpy="${math_pi_over_2} 0 ${math_pi_over_2}" xyz="0 0 0"/>
         <geometry>
-          <mesh filename="package://rb1_torso_description/meshes/sensors/asus_xtion_pro_live.dae" scale="0.001 0.001 0.001"/>
+          <mesh filename="package://rover_description/meshes/sensors/camera/asus_xtion_pro_live.dae" scale="0.001 0.001 0.001"/>
         </geometry>
       </collision>
