Commit message: masses fixed

File: rover_description/urdf/bases/bogie.urdf.xacro (robot description, xacro)
@@ -4,5 +4,5 @@
     <xacro:property name="bogie_box_width" value="0.29" />
     <xacro:property name="bogie_box_depth" value="0.10" />
-    <xacro:property name="bogie_box_mass" value="1.0" />
+    <xacro:property name="bogie_box_mass" value="0.25" />
     <xacro:include filename="$(find rover_description)/urdf/inertials.xacro"/>
     <xacro:macro name="bogie" params="lat_label reflect">

File: rover_description/urdf/bases/rocker.urdf.xacro (robot description, xacro)
@@ -4,5 +4,5 @@
     <xacro:property name="rocker_box_width" value="0.29" />
     <xacro:property name="rocker_box_depth" value="0.10" />
-    <xacro:property name="rocker_box_mass" value="1.0" />
+    <xacro:property name="rocker_box_mass" value="0.25" />
     <xacro:include filename="$(find rover_description)/urdf/inertials.xacro"/>
     <xacro:macro name="rocker" params="parent lat_label reflect">

File: rover_description/urdf/wheels/corner.urdf.xacro (robot description, xacro)
@@ -4,5 +4,5 @@
     <xacro:property name="corner_box_width" value="0.29" />
     <xacro:property name="corner_box_depth" value="0.10" />
-    <xacro:property name="corner_box_mass" value="1.0" />
+    <xacro:property name="corner_box_mass" value="0.25" />
     <xacro:include filename="$(find rover_description)/urdf/inertials.xacro"/>
     <!-- link -->

File: rover_description/urdf/wheels/wheel.urdf.xacro (robot description, xacro)
@@ -3,5 +3,5 @@
     <xacro:property name="wheel_width" value="0.100" />
     <xacro:property name="wheel_radius" value="0.060" />
-    <xacro:property name="wheel_mass" value="0.15" />
+    <xacro:property name="wheel_mass" value="0.25" />
     <xacro:include filename="$(find rover_description)/urdf/inertials.xacro"/>
     <!-- link -->
