Commit message: octomap

File: rover_description/urdf/bases/body.urdf.xacro (robot description, xacro)
@@ -30,5 +30,6 @@
                 <origin rpy="0 0 0" xyz="0 0 0" />
                 <geometry>
-                    <box size="${body_box_length} ${body_box_width} ${body_box_depth}"/>
+                    <mesh filename="package://rover_description/meshes/bases/body_box.stl" />
+                    <!-- <box size="${body_box_length} ${body_box_width} ${body_box_depth}"/> -->
                 </geometry>
             </collision>

File: rover_description/urdf/bases/rocker.urdf.xacro (robot description, xacro)
@@ -31,5 +31,6 @@
                 <origin rpy="0 0 0" xyz="0 0 0" />
                 <geometry>
-                    <box size="${rocker_box_length} ${rocker_box_width} ${rocker_box_depth}"/>
+                    <mesh filename="package://rover_description/meshes/bases/${lat_label}_rocker_asm.stl" />
+                    <!-- <box size="${rocker_box_length} ${rocker_box_width} ${rocker_box_depth}"/> -->
                 </geometry>
             </collision>

File: rover_description/urdf/sensors/hokuyo.urdf.xacro (robot description, xacro)
@@ -48,5 +48,5 @@
     </joint>
     <gazebo reference="${prefix}_link">
-            <sensor type="gpu_ray" name="hokuyo_sensor">
+            <sensor type="ray" name="hokuyo_sensor">
                 <pose>0 0 0 0 0 0</pose>
                 <visualize>true</visualize>
@@ -55,5 +55,5 @@
                     <scan>
                         <horizontal>
-                            <samples>1081</samples>
+                            <samples>30</samples>
                             <resolution>1</resolution>
                             <min_angle>${min_angle}</min_angle>

File: rover_description/urdf/wheels/corner.urdf.xacro (robot description, xacro)
@@ -31,5 +31,6 @@
                 <origin rpy="0 0 0" xyz="0 0 0" />
                 <geometry>
-                    <box size="${corner_box_length} ${corner_box_width} ${corner_box_depth}"/>
+                    <mesh filename="package://rover_description/meshes/bases/${lon_label}_${lat_label}_steering_asm.stl" />
+                    <!-- <box size="${corner_box_length} ${corner_box_width} ${corner_box_depth}"/> -->
                 </geometry>
             </collision>

Commit message: gpu_ray

File: rover_description/urdf/bases/body.urdf.xacro (robot description, xacro)
@@ -30,6 +30,6 @@
                 <origin rpy="0 0 0" xyz="0 0 0" />
                 <geometry>
-                    <mesh filename="package://rover_description/meshes/bases/body_box.stl" />
-                    <!-- <box size="${body_box_length} ${body_box_width} ${body_box_depth}"/> -->
+                    <!-- <mesh filename="package://rover_description/meshes/bases/body_box.stl" /> -->
+                    <box size="${body_box_length} ${body_box_width} ${body_box_depth}"/>
                 </geometry>
             </collision>

File: rover_description/urdf/bases/rocker.urdf.xacro (robot description, xacro)
@@ -31,6 +31,6 @@
                 <origin rpy="0 0 0" xyz="0 0 0" />
                 <geometry>
-                    <mesh filename="package://rover_description/meshes/bases/${lat_label}_rocker_asm.stl" />
-                    <!-- <box size="${rocker_box_length} ${rocker_box_width} ${rocker_box_depth}"/> -->
+                    <!-- <mesh filename="package://rover_description/meshes/bases/${lat_label}_rocker_asm.stl" /> -->
+                    <box size="${rocker_box_length} ${rocker_box_width} ${rocker_box_depth}"/>
                 </geometry>
             </collision>

File: rover_description/urdf/sensors/hokuyo.urdf.xacro (robot description, xacro)
@@ -48,5 +48,5 @@
     </joint>
     <gazebo reference="${prefix}_link">
-            <sensor type="ray" name="hokuyo_sensor">
+            <sensor type="gpu_ray" name="hokuyo_sensor">
                 <pose>0 0 0 0 0 0</pose>
                 <visualize>true</visualize>

File: rover_description/urdf/wheels/corner.urdf.xacro (robot description, xacro)
@@ -31,6 +31,6 @@
                 <origin rpy="0 0 0" xyz="0 0 0" />
                 <geometry>
-                    <mesh filename="package://rover_description/meshes/bases/${lon_label}_${lat_label}_steering_asm.stl" />
-                    <!-- <box size="${corner_box_length} ${corner_box_width} ${corner_box_depth}"/> -->
+                    <!-- <mesh filename="package://rover_description/meshes/bases/${lon_label}_${lat_label}_steering_asm.stl" /> -->
+                    <box size="${corner_box_length} ${corner_box_width} ${corner_box_depth}"/>
                 </geometry>
             </collision>
