Commit message: sensors fixed + moon world

File: rover_description/urdf/bases/rocker.urdf.xacro (robot description, xacro)
@@ -50,5 +50,5 @@
         </gazebo>
         <!-- joint -->
-        <joint name="${lat_label}_rocker_joint" type="continuous">
+        <joint name="${lat_label}_rocker_joint" type="fixed"> <!-- continuous -->
             <origin rpy="0 0 0" xyz="0.071 ${reflect * 0.155} 0.0118"/>
             <axis xyz="0 1 0" />

File: rover_description/urdf/sensors/asus_xtion.urdf.xacro (robot description, xacro)
@@ -48,5 +48,5 @@
     </link>
     <joint name="camera_frame_joint" type="fixed">
-      <origin xyz="0 0 0" rpy="-${math_pi_over_2} 0 -${math_pi_over_2}" />
+      <origin xyz="0 0 0" rpy="0 0 0" />
       <parent link="${prefix}_link" />
       <child link="camera_frame" />
@@ -63,4 +63,6 @@
     <gazebo reference="${prefix}_link">
       <sensor name="rgbd_camera" type="rgbd_camera">
+        <ignition_frame_id>camera_frame</ignition_frame_id>
+        <pose relative_to="camera_frame">0 0 0 0 0 0</pose>
         <camera>
           <horizontal_fov>1.3439</horizontal_fov>

File: rover_description/urdf/sensors/imu.urdf.xacro (robot description, xacro)
@@ -54,4 +54,6 @@
         <update_rate>200</update_rate>
         <visualize>true</visualize>
+        <ignition_frame_id>${prefix}_link</ignition_frame_id>
+        <pose relative_to="${prefix}_link">0 0 0 0 0 0</pose>
         <imu>
           <angular_velocity>
