Commit message: asus_xtion files renamed

File: rover_description/robots/rover.urdf.xacro (robot description, xacro)
@@ -66,7 +66,7 @@
         <origin xyz="0 0 -0.04" rpy="0 0 0"/>
     </xacro:sensor_imu>
-    <xacro:sennsor_depth_camera prefix="camera" parent="base_link">
+    <xacro:sensor_asus_xtion prefix="camera" parent="base_link">
         <origin xyz="0.212 0 0.065" rpy="0 0 0"/>
-    </xacro:sennsor_depth_camera>
+    </xacro:sensor_asus_xtion>
     <!-- wheels -->
     <xacro:corner_link lon_label="front" lat_label="left" reflect="1"/>

File: rover_description/urdf/sensors/all_sensors.urdf.xacro (robot description, xacro)
@@ -6,4 +6,4 @@
   <xacro:include filename="$(find rover_description)/urdf/sensors/hokuyo.urdf.xacro" />
   <!-- Hokuyo -->
-  <xacro:include filename="$(find rover_description)/urdf/sensors/depth_camera.urdf.xacro" />
+  <xacro:include filename="$(find rover_description)/urdf/sensors/asus_xtion.urdf.xacro" />
 </robot>

File: rover_description/urdf/sensors/asus_xtion.urdf.xacro (robot description, xacro)
@@ -1,5 +1,5 @@
 <?xml version="1.0"?>
-<robot name="sennsor_depth_camera" xmlns:xacro="http://www.ros.org/wiki/xacro">
-  <xacro:macro name="sennsor_depth_camera" params="prefix parent *origin ">
+<robot name="sensor_asus_xtion" xmlns:xacro="http://www.ros.org/wiki/xacro">
+  <xacro:macro name="sensor_asus_xtion" params="prefix parent *origin ">
     <xacro:property name="math_pi_over_2" value="1.5707963267948966" />
     <joint name="${prefix}_joint" type="fixed">
@@ -13,5 +13,5 @@
         <origin rpy="${math_pi_over_2} 0 ${math_pi_over_2}" xyz="0 0 0"/>
         <geometry>
-          <mesh filename="package://rover_description/meshes/sensors/camera/asus_xtion_pro_live.dae" scale="0.001 0.001 0.001"/>
+          <mesh filename="package://rover_description/meshes/sensors/asus_xtion/asus_xtion_pro_live.dae" scale="0.001 0.001 0.001"/>
         </geometry>
       </visual>
@@ -19,5 +19,5 @@
         <origin rpy="${math_pi_over_2} 0 ${math_pi_over_2}" xyz="0 0 0"/>
         <geometry>
-          <mesh filename="package://rover_description/meshes/sensors/camera/asus_xtion_pro_live.dae" scale="0.001 0.001 0.001"/>
+          <mesh filename="package://rover_description/meshes/sensors/asus_xtion/asus_xtion_pro_live.dae" scale="0.001 0.001 0.001"/>
         </geometry>
       </collision>

Commit message: tilted camera

File: rover_description/robots/rover.urdf.xacro (robot description, xacro)
@@ -67,5 +67,6 @@
     </xacro:sensor_imu>
     <xacro:sensor_asus_xtion prefix="camera" parent="base_link">
-        <origin xyz="0.212 0 0.065" rpy="0 0 0"/>
+        <origin xyz="0.215 0 0.065" rpy="0 0.5 0"/>
+        <!-- <origin xyz="0.212 0 0.065" rpy="0 0 0"/> -->
     </xacro:sensor_asus_xtion>
     <!-- wheels -->

Commit message: vault integration

File: rover_description/robots/rover.urdf.xacro (robot description, xacro)
@@ -11,5 +11,5 @@
     <xacro:include filename="$(find rover_description)/urdf/wheels/wheel.urdf.xacro" />
     <xacro:include filename="$(find rover_description)/urdf/wheels/corner.urdf.xacro" />
-    <xacro:include filename="$(find rover_description)/urdf/sensors/all_sensors.urdf.xacro" />
+    <xacro:include filename="$(find vault_description)/urdf/vault.urdf.xacro" />
     <!-- Gazebo ROS2 Control -->
     <gazebo>
@@ -58,16 +58,8 @@
     <xacro:bogie lat_label="left" reflect="1"/>
     <xacro:bogie lat_label="right" reflect="-1"/>
-    <!-- sensors -->
-    <xacro:sensor_hokuyo prefix="laser" parent="base_link" min_angle="-1.0" max_angle="1.0">
-        <origin xyz="0.17 0 0.005" rpy="0 0 0"/>
-    </xacro:sensor_hokuyo>
-    <xacro:sensor_imu prefix="imu" parent="base_link">
-        <!-- <origin xyz="-0.32 0 0.05" rpy="0 0.5 0"/> -->
-        <origin xyz="0 0 -0.04" rpy="0 0 0"/>
-    </xacro:sensor_imu>
-    <xacro:sensor_asus_xtion prefix="camera" parent="base_link">
-        <origin xyz="0.215 0 0.065" rpy="0 0.5 0"/>
-        <!-- <origin xyz="0.212 0 0.065" rpy="0 0 0"/> -->
-    </xacro:sensor_asus_xtion>
+    <!-- vault -->
+    <xacro:vault parent="base_link">
+        <origin xyz="0.1 0 0.05" rpy="0 0 0"/>
+    </xacro:vault>
     <!-- wheels -->
     <xacro:corner_link lon_label="front" lat_label="left" reflect="1"/>

Commit message: updates for humble

File: rover_description/robots/rover.urdf.xacro (robot description, xacro)
@@ -15,5 +15,5 @@
     <gazebo>
         <plugin filename="libgazebo_ros2_control.so" name="gazebo_ros2_control">
-        <parameters>$(find rover_description)/config/control.yaml</parameters>
+            <parameters>$(find rover_description)/config/control.yaml</parameters>
         </plugin>
     </gazebo>
@@ -30,10 +30,113 @@
             <joint_name>front_left_turnbuckle_joint</joint_name>
             <joint_name>front_right_turnbuckle_joint</joint_name>
+            <joint_name>front_left_corner_joint</joint_name>
+            <joint_name>front_right_corner_joint</joint_name>
             <joint_name>back_left_corner_joint</joint_name>
             <joint_name>back_right_corner_joint</joint_name>
-            <joint_name>front_left_corner_joint</joint_name>
-            <joint_name>front_right_corner_joint</joint_name>
         </plugin>
     </gazebo>
+    <ros2_control name="GazeboSystem" type="system">
+        <hardware>
+            <plugin>gazebo_ros2_control/GazeboSystem</plugin>
+        </hardware>
+        <joint name="front_right_corner_joint">
+            <command_interface name="position">
+                <param name="min">-3.14159</param>
+                <param name="max">3.14159</param>
+            </command_interface>
+            <state_interface name="position">
+                <param name="initial_value">0.0</param>
+            </state_interface>
+            <state_interface name="velocity"/>
+            <state_interface name="effort"/>
+        </joint>
+        <joint name="front_left_corner_joint">
+            <command_interface name="position">
+                <param name="min">-3.14159</param>
+                <param name="max">3.14159</param>
+            </command_interface>
+            <state_interface name="position">
+                <param name="initial_value">0.0</param>
+            </state_interface>
+            <state_interface name="velocity"/>
+            <state_interface name="effort"/>
+        </joint>
+        <joint name="back_right_corner_joint">
+            <command_interface name="position">
+                <param name="min">-3.14159</param>
+                <param name="max">3.14159</param>
+            </command_interface>
+            <state_interface name="position">
+                <param name="initial_value">0.0</param>
+            </state_interface>
+            <state_interface name="velocity"/>
+            <state_interface name="effort"/>
+        </joint>
+        <joint name="back_left_corner_joint">
+            <command_interface name="position">
+                <param name="min">-3.14159</param>
+                <param name="max">3.14159</param>
+            </command_interface>
+            <state_interface name="position">
+                <param name="initial_value">0.0</param>
+            </state_interface>
+            <state_interface name="velocity"/>
+            <state_interface name="effort"/>
+        </joint>
+        <joint name="front_right_wheel_joint">
+            <command_interface name="velocity">
+                <param name="min">-10</param>
+                <param name="max">10</param>
+            </command_interface>
+            <state_interface name="position"/>
+            <state_interface name="velocity"/>
+            <state_interface name="effort"/>
+        </joint>
+        <joint name="front_left_wheel_joint">
+            <command_interface name="velocity">
+                <param name="min">-10</param>
+                <param name="max">10</param>
+            </command_interface>
+            <state_interface name="position"/>
+            <state_interface name="velocity"/>
+            <state_interface name="effort"/>
+        </joint>
+        <joint name="mid_right_wheel_joint">
+            <command_interface name="velocity">
+                <param name="min">-10</param>
+                <param name="max">10</param>
+            </command_interface>
+            <state_interface name="position"/>
+            <state_interface name="velocity"/>
+            <state_interface name="effort"/>
+        </joint>
+        <joint name="mid_left_wheel_joint">
+            <command_interface name="velocity">
+                <param name="min">-10</param>
+                <param name="max">10</param>
+            </command_interface>
+            <state_interface name="position"/>
+            <state_interface name="velocity"/>
+            <state_interface name="effort"/>
+        </joint>
+        <joint name="back_right_wheel_joint">
+            <command_interface name="velocity">
+                <param name="min">-10</param>
+                <param name="max">10</param>
+            </command_interface>
+            <state_interface name="position"/>
+            <state_interface name="velocity"/>
+            <state_interface name="effort"/>
+        </joint>
+        <joint name="back_left_wheel_joint">
+            <command_interface name="velocity">
+                <param name="min">-10</param>
+                <param name="max">10</param>
+            </command_interface>
+            <state_interface name="position"/>
+            <state_interface name="velocity"/>
+            <state_interface name="effort"/>
+        </joint>
+    </ros2_control>
     <!-- The base link -->
     <link name="base_link">

File: rover_description/urdf/wheels/corner.urdf.xacro (robot description, xacro)
@@ -42,18 +42,4 @@
             <dynamics damping="0.0" friction="0.0"/>
         </joint>
-        <ros2_control name="GazeboSystem" type="system">
-            <hardware>
-                <plugin>gazebo_ros2_control/GazeboSystem</plugin>
-            </hardware>
-            <joint name="front_${lat_label}_corner_joint">
-            <command_interface name="position">
-                <param name="min">-3.14159</param>
-                <param name="max">3.14159</param>
-            </command_interface>
-            <state_interface name="position"/>
-            <state_interface name="velocity"/>
-            <state_interface name="effort"/>
-            </joint>
-        </ros2_control>
         <gazebo reference="front_${lat_label}_corner_joint">
             <provideFeedback>true</provideFeedback>
@@ -70,18 +56,4 @@
             <dynamics damping="0.0" friction="0.0"/>
         </joint>
-        <ros2_control name="GazeboSystem" type="system">
-            <hardware>
-                <plugin>gazebo_ros2_control/GazeboSystem</plugin>
-            </hardware>
-            <joint name="back_${lat_label}_corner_joint">
-            <command_interface name="position">
-                <param name="min">-3.14159</param>
-                <param name="max">3.14159</param>
-            </command_interface>
-            <state_interface name="position"/>
-            <state_interface name="velocity"/>
-            <state_interface name="effort"/>
-            </joint>
-        </ros2_control>
         <gazebo reference="back_${lat_label}_corner_joint">
             <provideFeedback>true</provideFeedback>

File: rover_description/urdf/wheels/wheel.urdf.xacro (robot description, xacro)
@@ -47,18 +47,4 @@
             <dynamics damping="0.0" friction="0.0"/>
         </joint>
-        <ros2_control name="GazeboSystem" type="system">
-            <hardware>
-                <plugin>gazebo_ros2_control/GazeboSystem</plugin>
-            </hardware>
-            <joint name="${lon_label}_${lat_label}_wheel_joint">
-                <command_interface name="velocity">
-                    <param name="min">-10</param>
-                    <param name="max">10</param>
-                </command_interface>
-                <state_interface name="position"/>
-                <state_interface name="velocity"/>
-                <state_interface name="effort"/>
-            </joint>
-        </ros2_control>
         <gazebo reference="${lon_label}_${lat_label}_wheel_joint">
             <provideFeedback>true</provideFeedback>
@@ -75,18 +61,4 @@
             <dynamics damping="0.0" friction="0.0"/>
         </joint>
-        <ros2_control name="GazeboSystem" type="system">
-            <hardware>
-                <plugin>gazebo_ros2_control/GazeboSystem</plugin>
-            </hardware>
-            <joint name="mid_${lat_label}_wheel_joint">
-                <command_interface name="velocity">
-                    <param name="min">-10</param>
-                    <param name="max">10</param>
-                </command_interface>
-                <state_interface name="position"/>
-                <state_interface name="velocity"/>
-                <state_interface name="effort"/>
-            </joint>
-        </ros2_control>
         <gazebo reference="mid_${lat_label}_wheel_joint">
             <provideFeedback>true</provideFeedback>

Commit message: camera fixed

File: rover_description/robots/rover.urdf.xacro (robot description, xacro)
@@ -181,5 +181,5 @@
     </xacro:sensor_imu>
     <xacro:sensor_asus_xtion prefix="camera" parent="base_link">
-        <origin xyz="0.215 0 0.065" rpy="0 0.5 0"/>
+        <origin xyz="0.215 0 0.065" rpy="0 0.2 0"/>
         <!-- <origin xyz="0.212 0 0.065" rpy="0 0 0"/> -->
     </xacro:sensor_asus_xtion>

File: rover_description/urdf/sensors/asus_xtion.urdf.xacro (robot description, xacro)
@@ -59,15 +59,22 @@
         <visualize>true</visualize>
         <update_rate>30</update_rate>
-        <camera name="depth_camera">
-          <horizontal_fov>1.3439</horizontal_fov>
+        <camera>
+          <horizontal_fov>${63.0*2*math_pi_over_2/180.0}</horizontal_fov>
           <image>
-            <width>720</width>
+            <format>B8G8R8</format>
+            <width>640</width>
             <height>480</height>
-            <format>R8G8B8</format>
           </image>
           <clip>
-            <near>0.05</near>
-            <far>3</far>
+            <near>0.3</near>
+            <far>8.0</far>
           </clip>
+	        <distortion>
+            <k1>0.00000001</k1>
+            <k2>0.00000001</k2>
+            <k3>0.00000001</k3>
+            <p1>0.00000001</p1>
+            <p2>0.00000001</p2>
+          </distortion>
         </camera>
         <plugin name="depth_camera_controller" filename="libgazebo_ros_camera.so">
@@ -131,20 +138,7 @@
             </qos>
           </ros>
-          <baseline>0.2</baseline>
-          <always_on>true</always_on>
-          <update_rate>0.0</update_rate>
           <frame_name>camera_frame</frame_name>
-          <point_cloud_cutoff>0.5</point_cloud_cutoff>
-          <point_cloud_cutoff_max>3.0</point_cloud_cutoff_max>
-          <distortion_k1>0</distortion_k1>
-          <distortion_k2>0</distortion_k2>
-          <distortion_k3>0</distortion_k3>
-          <distortion_t1>0</distortion_t1>
-          <distortion_t2>0</distortion_t2>
-          <CxPrime>0</CxPrime>
-          <Cx>0</Cx>
-          <Cy>0</Cy>
-          <focal_length>0</focal_length>
-          <hack_baseline>0</hack_baseline>
+          <min_depth>0.3</min_depth>
+          <max_depth>8.0</max_depth>
         </plugin>
       </sensor>

Commit message: gazebo fixes

File: rover_description/robots/rover.urdf.xacro (robot description, xacro)
@@ -181,5 +181,5 @@
     </xacro:sensor_imu>
     <xacro:sensor_asus_xtion prefix="camera" parent="base_link">
-        <origin xyz="0.215 0 0.065" rpy="0 0.2 0"/>
+        <origin xyz="0.215 0 0.065" rpy="0 0.4 0"/>
         <!-- <origin xyz="0.212 0 0.065" rpy="0 0 0"/> -->
     </xacro:sensor_asus_xtion>
