Commit message: initial changes for ignition

File: rover_description/robots/rover.urdf.xacro (robot description, xacro)
@@ -31,29 +31,21 @@
     <!-- Gazebo ROS2 Control -->
     <gazebo>
-        <plugin filename="libgazebo_ros2_control.so" name="gazebo_ros2_control">
-            <parameters>$(find rover_description)/config/control.yaml</parameters>
+        <plugin filename="libign_ros2_control-system.so" name="ign_ros2_control::IgnitionROS2ControlPlugin">
+        <parameters>$(find rover_description)/config/control.yaml</parameters>
+        <ros>
+            <remapping>/tf:=tf</remapping>
+            <remapping>/tf_static:=tf_static</remapping>
+        </ros>
+        </plugin>
+        <plugin filename="libignition-gazebo-sensors-system.so" name="ignition::gazebo::systems::Sensors">
+        <render_engine>ogre2</render_engine>
+        </plugin>
+        <plugin filename="libignition-gazebo-imu-system.so"
+                name="ignition::gazebo::systems::Imu">
         </plugin>
     </gazebo>
-    <gazebo>
-        <plugin name="rover_joint_state" filename="libgazebo_ros_joint_state_publisher.so">
-            <update_rate>30</update_rate>
-            <joint_name>left_rocker_joint</joint_name>
-            <joint_name>right_rocker_joint</joint_name>
-            <joint_name>left_bogie_joint</joint_name>
-            <joint_name>right_bogie_joint</joint_name>
-            <joint_name>diff_brace_joint</joint_name>
-            <joint_name>back_left_turnbuckle_joint</joint_name>
-            <joint_name>back_right_turnbuckle_joint</joint_name>
-            <joint_name>front_left_turnbuckle_joint</joint_name>
-            <joint_name>front_right_turnbuckle_joint</joint_name>
-            <joint_name>front_left_corner_joint</joint_name>
-            <joint_name>front_right_corner_joint</joint_name>
-            <joint_name>back_left_corner_joint</joint_name>
-            <joint_name>back_right_corner_joint</joint_name>
-        </plugin>
-    </gazebo>
-    <ros2_control name="GazeboSystem" type="system">
+    <ros2_control name="IgnitionSystem" type="system">
         <hardware>
-            <plugin>gazebo_ros2_control/GazeboSystem</plugin>
+            <plugin>ign_ros2_control/IgnitionSystem</plugin>
         </hardware>
         <joint name="front_right_corner_joint">
@@ -172,6 +164,6 @@
     <xacro:body parent="base_link" />
     <xacro:differential parent="base_link" />
-    <xacro:turnbuckle lat_label="left" reflect="1"/>
-    <xacro:turnbuckle lat_label="right" reflect="-1"/>
+    <!-- <xacro:turnbuckle lat_label="left" reflect="1"/>
+    <xacro:turnbuckle lat_label="right" reflect="-1"/> -->
     <xacro:rocker parent="base_link" lat_label="left" reflect="1"/>
     <xacro:rocker parent="base_link" lat_label="right" reflect="-1"/>

File: rover_description/urdf/bases/body.urdf.xacro (robot description, xacro)
@@ -17,5 +17,5 @@
 # OUT OF OR IN CONNECTION WITH THE SOFTWARE OR THE USE OR OTHER DEALINGS IN THE
 # SOFTWARE. -->
-<robot name="body" xmlns:xacro="http://www.ros.org/wiki/xacro">
+<robot xmlns:xacro="http://www.ros.org/wiki/xacro">
     <xacro:property name="body_box_length" value="0.43" />
     <xacro:property name="body_box_width" value="0.29" />

File: rover_description/urdf/bases/bogie.urdf.xacro (robot description, xacro)
@@ -17,5 +17,5 @@
 # OUT OF OR IN CONNECTION WITH THE SOFTWARE OR THE USE OR OTHER DEALINGS IN THE
 # SOFTWARE. -->
-<robot name="rocker" xmlns:xacro="http://www.ros.org/wiki/xacro">
+<robot xmlns:xacro="http://www.ros.org/wiki/xacro">
     <xacro:property name="bogie_box_length" value="0.43" />
     <xacro:property name="bogie_box_width" value="0.29" />
@@ -60,8 +60,4 @@
             <child link="${lat_label}_bogie_link" />
         </joint>
-        <gazebo reference="${lat_label}_bogie_joint">
-            <provideFeedback>true</provideFeedback>
-            <implicitSpringDamper>true</implicitSpringDamper>
-        </gazebo>
     </xacro:macro>
 </robot>

File: rover_description/urdf/bases/differential.urdf.xacro (robot description, xacro)
@@ -17,5 +17,5 @@
 # OUT OF OR IN CONNECTION WITH THE SOFTWARE OR THE USE OR OTHER DEALINGS IN THE
 # SOFTWARE. -->
-<robot name="differential" xmlns:xacro="http://www.ros.org/wiki/xacro">
+<robot xmlns:xacro="http://www.ros.org/wiki/xacro">
     <xacro:property name="differential_box_length" value="0.300" />
     <xacro:property name="differential_box_width" value="0.055" />
@@ -59,8 +59,4 @@
             <child link="diff_brace_link" />
         </joint>
-        <gazebo reference="diff_brace_joint">
-            <provideFeedback>true</provideFeedback>
-            <implicitSpringDamper>true</implicitSpringDamper>
-        </gazebo>
     </xacro:macro>
 </robot>

File: rover_description/urdf/bases/rocker.urdf.xacro (robot description, xacro)
@@ -17,5 +17,5 @@
 # OUT OF OR IN CONNECTION WITH THE SOFTWARE OR THE USE OR OTHER DEALINGS IN THE
 # SOFTWARE. -->
-<robot name="rocker" xmlns:xacro="http://www.ros.org/wiki/xacro">
+<robot xmlns:xacro="http://www.ros.org/wiki/xacro">
     <xacro:property name="rocker_box_length" value="0.43" />
     <xacro:property name="rocker_box_width" value="0.29" />

File: rover_description/urdf/bases/turnbuckle.urdf.xacro (robot description, xacro)
@@ -17,59 +17,48 @@
 # OUT OF OR IN CONNECTION WITH THE SOFTWARE OR THE USE OR OTHER DEALINGS IN THE
 # SOFTWARE. -->
-<robot name="turnbuckle" xmlns:xacro="http://www.ros.org/wiki/xacro">
+<robot xmlns:xacro="http://www.ros.org/wiki/xacro">
     <xacro:include filename="$(find rover_description)/urdf/inertials.xacro"/>
     <xacro:macro name="turnbuckle" params="lat_label reflect">
-        <gazebo>
             <link name="${lat_label}_turnbuckle_link">
-                <pose>0.035 ${reflect * 0.17} 0.07 0 0 0</pose>
-                <visual name="${lat_label}_turnbuckle_visual">
-                    <pose>0 0 0 0 0 0</pose>
+                <origin xyz="0.035 ${reflect * 0.17} 0.07" rpy="0 0 0"/>
+                <visual>
+                    <origin rpy="0 0 0" xyz="0 0 0" />
                     <geometry>
-                        <mesh>
-                            <uri>package://rover_description/meshes/bases/turnbuckle.stl</uri>
-                        </mesh>
-                        <!-- <cylinder>
-                            <length>0.07</length>
-                            <radius>0.0025</radius>
-                        </cylinder> -->
+                        <mesh filename="package://rover_description/meshes/bases/turnbuckle.stl" />
                     </geometry>
-                    <material>
-                        <script>
-                            <name>Gazebo/Blue</name>
-                        </script>
-                    </material>
+                    <material name="blue" />
                 </visual>
-                <collision name="${lat_label}_turnbuckle_collision">
-                    <pose>0 0 0 0 ${math_pi_over_2} 0</pose>
+                <collision>
+                    <origin xyz="0 0 0" rpy="0 ${math_pi_over_2} 0"/>
                     <geometry>
-                        <cylinder>
-                            <length>0.07</length>
-                            <radius>0.0025</radius>
-                        </cylinder>
+                        <cylinder length="0.07" radius="0.0025"/>
                     </geometry>
                 </collision>
-                <inertial>
-                    <mass>0.01</mass>
-                    <inertia>
-                        <ixx>0.0001</ixx>
-                        <ixy>0</ixy>
-                        <ixz>0</ixz>
-                        <iyy>0.0001</iyy>
-                        <iyz>0</iyz>
-                        <izz>0.0001</izz>
-                    </inertia>
-                </inertial>
+                <xacro:solid_cylinder_inertial
+                    rpy="0 0 0" xyz="0 0 0"
+                    mass="0.25"
+                    radius="0.0025"
+                    length="0.07" />
             </link>
-            <joint name="back_${lat_label}_turnbuckle_joint" type="ball">
-                <pose>-0.035 0 0 0 0 0</pose>
-                <parent>diff_brace_link</parent>
-                <child>${lat_label}_turnbuckle_link</child>
+            <joint name="back_${lat_label}_turnbuckle_joint" type="revolute">
+                <origin xyz="-0.035 0 0" rpy="0 0 0"/>
+                <limit
+                    lower="${-math_pi}"
+                    upper="${math_pi}"
+                    effort="100.0"
+                    velocity="30.0" />
+                <parent link="diff_brace_link" />
+                <child link="${lat_label}_turnbuckle_link" />
             </joint>
-            <joint name="front_${lat_label}_turnbuckle_joint" type="ball">
-                <pose>0.035 0 0 0 0 0</pose>
-                <parent>${lat_label}_rocker_link</parent>
-                <child>${lat_label}_turnbuckle_link</child>
-            </joint>
-        </gazebo>
+            <!-- <joint name="front_${lat_label}_turnbuckle_joint" type="revolute">
+                <origin xyz="0.035 0 0" rpy="0 0 0"/>
+                <limit
+                    lower="${-math_pi}"
+                    upper="${math_pi}"
+                    effort="100.0"
+                    velocity="30.0" />
+                <parent link="${lat_label}_rocker_link" />
+                <child link="${lat_label}_turnbuckle_link" />
+            </joint> -->
     </xacro:macro>
 </robot>

File: rover_description/urdf/sensors/asus_xtion.urdf.xacro (robot description, xacro)
@@ -17,5 +17,5 @@
 # OUT OF OR IN CONNECTION WITH THE SOFTWARE OR THE USE OR OTHER DEALINGS IN THE
 # SOFTWARE. -->
-<robot name="sensor_asus_xtion" xmlns:xacro="http://www.ros.org/wiki/xacro">
+<robot xmlns:xacro="http://www.ros.org/wiki/xacro">
   <xacro:macro name="sensor_asus_xtion" params="prefix parent *origin ">
     <xacro:property name="math_pi_over_2" value="1.5707963267948966" />
@@ -62,90 +62,22 @@
     </link>
     <gazebo reference="${prefix}_link">
-      <sensor name="camera" type="depth">
-        <visualize>true</visualize>
-        <update_rate>30</update_rate>
+      <sensor name="rgbd_camera" type="rgbd_camera">
         <camera>
-          <horizontal_fov>${63.0*2*math_pi_over_2/180.0}</horizontal_fov>
+          <horizontal_fov>1.3439</horizontal_fov>
           <image>
-            <format>B8G8R8</format>
-            <width>640</width>
+            <width>720</width>
             <height>480</height>
+            <format>R8G8B8</format>
           </image>
           <clip>
-            <near>0.3</near>
-            <far>8.0</far>
+            <near>0.05</near>
+            <far>100</far>
           </clip>
-	        <distortion>
-            <k1>0.00000001</k1>
-            <k2>0.00000001</k2>
-            <k3>0.00000001</k3>
-            <p1>0.00000001</p1>
-            <p2>0.00000001</p2>
-          </distortion>
+          <optical_frame_id>camera_frame</optical_frame_id>
         </camera>
-        <plugin name="depth_camera_controller" filename="libgazebo_ros_camera.so">
-          <ros>
-            <qos>
-              <topic name="/camera/camera_info">
-                <publisher>
-                  <reliability>best_effort</reliability>
-                </publisher>
-              </topic>
-              <topic name="/camera/image_raw">
-                <publisher>
-                  <reliability>best_effort</reliability>
-                </publisher>
-              </topic>
-              <topic name="/camera/image_raw/compressed">
-                <publisher>
-                  <reliability>best_effort</reliability>
-                </publisher>
-              </topic>
-              <topic name="/camera/image_raw/compressedDepth">
-                <publisher>
-                  <reliability>best_effort</reliability>
-                </publisher>
-              </topic>
-              <topic name="/camera/image_raw/theora">
-                <publisher>
-                  <reliability>best_effort</reliability>
-                </publisher>
-              </topic>
-              <topic name="/camera/points">
-                <publisher>
-                  <reliability>best_effort</reliability>
-                </publisher>
-              </topic>
-              <topic name="/camera/depth/camera_info">
-                <publisher>
-                  <reliability>best_effort</reliability>
-                </publisher>
-              </topic>
-              <topic name="/camera/depth/image_raw">
-                <publisher>
-                  <reliability>best_effort</reliability>
-                </publisher>
-              </topic>
-              <topic name="/camera/depth/image_raw/compressed">
-                <publisher>
-                  <reliability>best_effort</reliability>
-                </publisher>
-              </topic>
-              <topic name="/camera/depth/image_raw/compressedDepth">
-                <publisher>
-                  <reliability>best_effort</reliability>
-                </publisher>
-              </topic>
-             <topic name="/camera/depth/image_raw/theora">
-                <publisher>
-                  <reliability>best_effort</reliability>
-                </publisher>
-              </topic>
-            </qos>
-          </ros>
-          <frame_name>camera_frame</frame_name>
-          <min_depth>0.3</min_depth>
-          <max_depth>8.0</max_depth>
-        </plugin>
+        <always_on>1</always_on>
+        <topic>camera</topic>
+        <update_rate>30</update_rate>
+        <visualize>true</visualize>
       </sensor>
     </gazebo>

File: rover_description/urdf/sensors/hokuyo.urdf.xacro (robot description, xacro)
@@ -17,5 +17,5 @@
 # OUT OF OR IN CONNECTION WITH THE SOFTWARE OR THE USE OR OTHER DEALINGS IN THE
 # SOFTWARE. -->
-<robot name="sensor_hokuyo" xmlns:xacro="http://www.ros.org/wiki/xacro">
+<robot xmlns:xacro="http://www.ros.org/wiki/xacro">
   <xacro:macro name="sensor_hokuyo" params="prefix parent *origin min_angle:=-1.57079637051 max_angle:=1.57079637051">
     <joint name="${prefix}_base_joint" type="fixed">
@@ -54,43 +54,33 @@
     </joint>
     <gazebo reference="${prefix}_link">
-            <sensor type="gpu_ray" name="hokuyo_sensor">
-                <pose>0 0 0 0 0 0</pose>
-                <visualize>true</visualize>
-                <update_rate>50</update_rate>
-                <ray>
-                    <scan>
-                        <horizontal>
-                            <samples>30</samples>
-                            <resolution>1</resolution>
-                            <min_angle>${min_angle}</min_angle>
-                            <max_angle>${max_angle}</max_angle>
-                        </horizontal>
-                    </scan>
-                    <range>
-                        <min>0.06</min>
-                        <max>5.0</max>
-                        <resolution>0.004359297</resolution>
-                    </range>
-                    <noise>
-                        <type>gaussian</type>
-                        <mean>0.0</mean>
-                        <stddev>0.01</stddev>
-                    </noise>
-                </ray>
-                <plugin name="${prefix}_controller" filename="libgazebo_ros_ray_sensor.so">
-                  <ros>
-                    <remapping>~/out:=scan</remapping>
-                    <qos>
-                      <topic name="scan">
-                        <publisher>
-                          <reliability>best_effort</reliability>
-                        </publisher>
-                      </topic>
-                    </qos>
-                  </ros>
-                  <output_type>sensor_msgs/LaserScan</output_type>
-                  <frame_name>${prefix}_link</frame_name>
-                </plugin>
-            </sensor>
+        <sensor name="lidar" type="gpu_lidar">"
+            <ignition_frame_id>${prefix}_link</ignition_frame_id>
+            <pose relative_to="${prefix}_link">0 0 0 0 0 0</pose>
+            <topic>/scan</topic>
+            <update_rate>10</update_rate>
+            <ray>
+                <scan>
+                    <horizontal>
+                        <samples>1081</samples>
+                        <resolution>1</resolution>
+                        <min_angle>${min_angle}</min_angle>
+                        <max_angle>${max_angle}</max_angle>
+                    </horizontal>
+                    <vertical>
+                        <samples>1</samples>
+                        <resolution>0.01</resolution>
+                        <min_angle>0</min_angle>
+                        <max_angle>0</max_angle>
+                    </vertical>
+                </scan>
+                <range>
+                    <min>0.06</min>
+                    <max>5.0</max>
+                    <resolution>0.01</resolution>
+                </range>
+            </ray>
+            <always_on>1</always_on>
+            <visualize>true</visualize>
+        </sensor>
     </gazebo>
   </xacro:macro>

File: rover_description/urdf/sensors/imu.urdf.xacro (robot description, xacro)
@@ -17,5 +17,5 @@
 # OUT OF OR IN CONNECTION WITH THE SOFTWARE OR THE USE OR OTHER DEALINGS IN THE
 # SOFTWARE. -->
-<robot name="sensor_imu" xmlns:xacro="http://www.ros.org/wiki/xacro">
+<robot xmlns:xacro="http://www.ros.org/wiki/xacro">
   <xacro:macro name="sensor_imu" params="prefix parent *origin">
     <joint name="${prefix}_joint" type="fixed">
@@ -50,19 +50,6 @@
     <gazebo reference="${prefix}_link">
       <sensor name="imu_sensor" type="imu">
-        <plugin filename="libgazebo_ros_imu_sensor.so" name="imu_controller">
-          <ros>
-            <remapping>~/out:=imu</remapping>
-            <qos>
-              <topic name="imu">
-                <publisher>
-                  <reliability>best_effort</reliability>
-                </publisher>
-              </topic>
-            </qos>
-          </ros>
-          <initial_orientation_as_reference>false</initial_orientation_as_reference>
-          <frame_name>${prefix}_link</frame_name>
-        </plugin>
-        <always_on>true</always_on>
+        <topic>imu</topic>
+        <always_on>1</always_on>
         <update_rate>200</update_rate>
         <visualize>true</visualize>

File: rover_description/urdf/wheels/corner.urdf.xacro (robot description, xacro)
@@ -17,5 +17,5 @@
 # OUT OF OR IN CONNECTION WITH THE SOFTWARE OR THE USE OR OTHER DEALINGS IN THE
 # SOFTWARE. -->
-<robot name="corner" xmlns:xacro="http://www.ros.org/wiki/xacro">
+<robot xmlns:xacro="http://www.ros.org/wiki/xacro">
     <xacro:property name="corner_box_length" value="0.43" />
     <xacro:property name="corner_box_width" value="0.29" />

File: rover_description/urdf/wheels/wheel.urdf.xacro (robot description, xacro)
@@ -17,5 +17,5 @@
 # OUT OF OR IN CONNECTION WITH THE SOFTWARE OR THE USE OR OTHER DEALINGS IN THE
 # SOFTWARE. -->
-<robot name="body" xmlns:xacro="http://www.ros.org/wiki/xacro">
+<robot xmlns:xacro="http://www.ros.org/wiki/xacro">
     <xacro:property name="wheel_width" value="0.100" />
     <xacro:property name="wheel_radius" value="0.060" />
