Commit message: fixing code format

File: rover_description/robots/rover.urdf.xacro (robot description, xacro)
@@ -17,5 +17,6 @@
 # OUT OF OR IN CONNECTION WITH THE SOFTWARE OR THE USE OR OTHER DEALINGS IN THE
 # SOFTWARE. -->
-<robot name="rover" xmlns:xacro="http://www.ros.org/wiki/xacro">
+<robot name="rover"
+    xmlns:xacro="http://www.ros.org/wiki/xacro">
     <!-- Include macros -->
     <xacro:include filename="$(find rover_description)/urdf/materials.xacro"/>
@@ -31,15 +32,14 @@
     <gazebo>
         <plugin filename="gz_ros2_control-system" name="gz_ros2_control::GazeboSimROS2ControlPlugin">
-        <parameters>$(find rover_description)/config/control.yaml</parameters>
-        <ros>
-            <remapping>/tf:=tf</remapping>
-            <remapping>/tf_static:=tf_static</remapping>
-        </ros>
+            <parameters>$(find rover_description)/config/control.yaml</parameters>
+            <ros>
+                <remapping>/tf:=tf</remapping>
+                <remapping>/tf_static:=tf_static</remapping>
+            </ros>
         </plugin>
         <plugin filename="libignition-gazebo-sensors-system.so" name="ignition::gazebo::systems::Sensors">
-        <render_engine>ogre2</render_engine>
+            <render_engine>ogre2</render_engine>
         </plugin>
-        <plugin filename="libignition-gazebo-imu-system.so"
-                name="ignition::gazebo::systems::Imu">
+        <plugin filename="libignition-gazebo-imu-system.so" name="ignition::gazebo::systems::Imu">
         </plugin>
     </gazebo>

File: rover_description/urdf/bases/body.urdf.xacro (robot description, xacro)
@@ -40,8 +40,5 @@
                 </geometry>
             </collision>
-            <xacro:solid_cuboid_inertial
-                rpy="0 0 0" xyz="0 0 0"
-                mass="${body_box_mass}"
-                x="${body_box_length}" y="${body_box_width}" z="${body_box_depth}" />
+            <xacro:solid_cuboid_inertial rpy="0 0 0" xyz="0 0 0" mass="${body_box_mass}" x="${body_box_length}" y="${body_box_width}" z="${body_box_depth}" />
         </link>
         <gazebo reference="body_box_link">

File: rover_description/urdf/bases/bogie.urdf.xacro (robot description, xacro)
@@ -40,8 +40,5 @@
                 </geometry>
             </collision>
-            <xacro:solid_cuboid_inertial
-                rpy="0 0 0" xyz="0 0 0"
-                mass="${bogie_box_mass}"
-                x="${bogie_box_length}" y="${bogie_box_width}" z="${bogie_box_depth}" />
+            <xacro:solid_cuboid_inertial rpy="0 0 0" xyz="0 0 0" mass="${bogie_box_mass}" x="${bogie_box_length}" y="${bogie_box_width}" z="${bogie_box_depth}" />
         </link>
         <gazebo reference="${lat_label}_bogie_link">
@@ -52,9 +49,5 @@
             <origin rpy="0 0 0" xyz="-0.181 ${reflect * 0.025} -0.062"/>
             <axis xyz="0 1 0" />
-            <limit
-                lower="${-math_pi_over_4}"
-                upper="${math_pi_over_4}"
-                effort="100.0"
-                velocity="30.0" />
+            <limit lower="${-math_pi_over_4}" upper="${math_pi_over_4}" effort="100.0" velocity="30.0" />
             <parent link="${lat_label}_rocker_link" />
             <child link="${lat_label}_bogie_link" />

File: rover_description/urdf/bases/differential.urdf.xacro (robot description, xacro)
@@ -40,8 +40,5 @@
                 </geometry>
             </collision>
-            <xacro:solid_cuboid_inertial
-                rpy="0 0 ${math_pi_over_2}" xyz="0 0 0"
-                mass="${differential_box_mass}"
-                x="${differential_box_length}" y="${differential_box_width}" z="${differential_box_depth}" />
+            <xacro:solid_cuboid_inertial rpy="0 0 ${math_pi_over_2}" xyz="0 0 0" mass="${differential_box_mass}" x="${differential_box_length}" y="${differential_box_width}" z="${differential_box_depth}" />
         </link>
         <gazebo reference="diff_brace_link">
@@ -51,9 +48,5 @@
             <origin rpy="0 0 0" xyz="0 0 0.0681"/>
             <axis xyz="0 0 1" />
-            <limit
-                lower="${-math_pi_over_4}"
-                upper="${math_pi_over_4}"
-                effort="100.0"
-                velocity="30.0" />
+            <limit lower="${-math_pi_over_4}" upper="${math_pi_over_4}" effort="100.0" velocity="30.0" />
             <parent link="${parent}" />
             <child link="diff_brace_link" />

File: rover_description/urdf/bases/rocker.urdf.xacro (robot description, xacro)
@@ -41,8 +41,5 @@
                 </geometry>
             </collision>
-            <xacro:solid_cuboid_inertial
-                rpy="0 0 0" xyz="0 0 0"
-                mass="${rocker_box_mass}"
-                x="${rocker_box_length}" y="${rocker_box_width}" z="${rocker_box_depth}" />
+            <xacro:solid_cuboid_inertial rpy="0 0 0" xyz="0 0 0" mass="${rocker_box_mass}" x="${rocker_box_length}" y="${rocker_box_width}" z="${rocker_box_depth}" />
         </link>
         <gazebo reference="${lat_label}_rocker_link">
@@ -50,12 +47,8 @@
         </gazebo>
         <!-- joint -->
-        <joint name="${lat_label}_rocker_joint" type="fixed"> <!-- continuous -->
+        <joint name="${lat_label}_rocker_joint" type="fixed">            <!-- continuous -->
             <origin rpy="0 0 0" xyz="0.071 ${reflect * 0.155} 0.0118"/>
             <axis xyz="0 1 0" />
-            <limit
-                lower="${-math_pi_over_4}"
-                upper="${math_pi_over_4}"
-                effort="100.0"
-                velocity="30.0" />
+            <limit lower="${-math_pi_over_4}" upper="${math_pi_over_4}" effort="100.0" velocity="30.0" />
             <parent link="${parent}" />
             <child link="${lat_label}_rocker_link" />

File: rover_description/urdf/bases/turnbuckle.urdf.xacro (robot description, xacro)
@@ -20,42 +20,30 @@
     <xacro:include filename="$(find rover_description)/urdf/inertials.xacro"/>
     <xacro:macro name="turnbuckle" params="lat_label reflect">
-            <link name="${lat_label}_turnbuckle_link">
-                <origin xyz="0.035 ${reflect * 0.17} 0.07" rpy="0 0 0"/>
-                <visual>
-                    <origin rpy="0 0 0" xyz="0 0 0" />
-                    <geometry>
-                        <mesh filename="package://rover_description/meshes/bases/turnbuckle.stl" />
-                    </geometry>
-                    <material name="blue" />
-                </visual>
-                <collision>
-                    <origin xyz="0 0 0" rpy="0 ${math_pi_over_2} 0"/>
-                    <geometry>
-                        <cylinder length="0.07" radius="0.0025"/>
-                    </geometry>
-                </collision>
-                <xacro:solid_cylinder_inertial
-                    rpy="0 0 0" xyz="0 0 0"
-                    mass="0.25"
-                    radius="0.0025"
-                    length="0.07" />
-            </link>
-            <joint name="back_${lat_label}_turnbuckle_joint" type="revolute">
-                <origin xyz="-0.035 0 0" rpy="0 0 0"/>
-                <limit
-                    lower="${-math_pi}"
-                    upper="${math_pi}"
-                    effort="100.0"
-                    velocity="30.0" />
-                <parent link="diff_brace_link" />
-                <child link="${lat_label}_turnbuckle_link" />
-            </joint>
-            <!-- <joint name="front_${lat_label}_turnbuckle_joint" type="revolute">
+        <link name="${lat_label}_turnbuckle_link">
+            <origin xyz="0.035 ${reflect * 0.17} 0.07" rpy="0 0 0"/>
+            <visual>
+                <origin rpy="0 0 0" xyz="0 0 0" />
+                <geometry>
+                    <mesh filename="package://rover_description/meshes/bases/turnbuckle.stl" />
+                </geometry>
+                <material name="blue" />
+            </visual>
+            <collision>
+                <origin xyz="0 0 0" rpy="0 ${math_pi_over_2} 0"/>
+                <geometry>
+                    <cylinder length="0.07" radius="0.0025"/>
+                </geometry>
+            </collision>
+            <xacro:solid_cylinder_inertial rpy="0 0 0" xyz="0 0 0" mass="0.25" radius="0.0025" length="0.07" />
+        </link>
+        <joint name="back_${lat_label}_turnbuckle_joint" type="revolute">
+            <origin xyz="-0.035 0 0" rpy="0 0 0"/>
+            <limit lower="${-math_pi}" upper="${math_pi}" effort="100.0" velocity="30.0" />
+            <parent link="diff_brace_link" />
+            <child link="${lat_label}_turnbuckle_link" />
+        </joint>
+        <!-- <joint name="front_${lat_label}_turnbuckle_joint" type="revolute">
                 <origin xyz="0.035 0 0" rpy="0 0 0"/>
-                <limit
-                    lower="${-math_pi}"
-                    upper="${math_pi}"
-                    effort="100.0"
-                    velocity="30.0" />
+                <limit lower="${-math_pi}" upper="${math_pi}" effort="100.0" velocity="30.0" />
                 <parent link="${lat_label}_rocker_link" />
                 <child link="${lat_label}_turnbuckle_link" />

File: rover_description/urdf/inertials.xacro (robot description, xacro)
@@ -17,7 +17,8 @@
 # OUT OF OR IN CONNECTION WITH THE SOFTWARE OR THE USE OR OTHER DEALINGS IN THE
 # SOFTWARE. -->
-<robot name="inertials" xmlns:xacro="http://www.ros.org/wiki/xacro">
+<robot name="inertials"
+    xmlns:xacro="http://www.ros.org/wiki/xacro">
     <!-- Math constants -->
-    <xacro:property name="math_pi"        value="3.141592653589793" />
+    <xacro:property name="math_pi" value="3.141592653589793" />
     <xacro:property name="math_pi_over_2" value="1.5707963267948966" />
     <xacro:property name="math_pi_over_4" value="0.785398163397448" />
@@ -27,8 +28,5 @@
             <origin rpy="${rpy}" xyz="${xyz}"/>
             <mass value="${mass}" />
-            <inertia
-                ixx="${mass * (y * y + z * z) / 12.0}" ixy="0.0" ixz="0.0"
-                iyy="${mass * (x * x + z * z) / 12.0}" iyz="0.0"
-                izz="${mass * (x * x + y * y) / 12.0}" />
+            <inertia ixx="${mass * (y * y + z * z) / 12.0}" ixy="0.0" ixz="0.0" iyy="${mass * (x * x + z * z) / 12.0}" iyz="0.0" izz="${mass * (x * x + y * y) / 12.0}" />
         </inertial>
     </xacro:macro>
@@ -38,8 +36,5 @@
             <origin rpy="${rpy}" xyz="${xyz}"/>
             <mass value="${mass}" />
-            <inertia
-                ixx="${mass * (3.0 * radius * radius + length * length) / 12.0}" ixy="0.0" ixz="0.0"
-                iyy="${mass * (3.0 * radius * radius + length * length) / 12.0}" iyz="0.0"
-                izz="${mass * (radius * radius) / 2.0}" />
+            <inertia ixx="${mass * (3.0 * radius * radius + length * length) / 12.0}" ixy="0.0" ixz="0.0" iyy="${mass * (3.0 * radius * radius + length * length) / 12.0}" iyz="0.0" izz="${mass * (radius * radius) / 2.0}" />
         </inertial>
     </xacro:macro>

File: rover_description/urdf/materials.xacro (robot description, xacro)
@@ -17,6 +17,7 @@
 # OUT OF OR IN CONNECTION WITH THE SOFTWARE OR THE USE OR OTHER DEALINGS IN THE
 # SOFTWARE. -->
-<robot name="materials" xmlns:xacro="http://www.ros.org/wiki/xacro">
-   <material name="red">
+<robot name="materials"
+    xmlns:xacro="http://www.ros.org/wiki/xacro">
+    <material name="red">
         <color rgba="0.8 0 0 1"/>
     </material>

File: rover_description/urdf/sensors/all_sensors.urdf.xacro (robot description, xacro)
@@ -17,5 +17,6 @@
 # OUT OF OR IN CONNECTION WITH THE SOFTWARE OR THE USE OR OTHER DEALINGS IN THE
 # SOFTWARE. -->
-<robot name="all_sensors" xmlns:xacro="http://www.ros.org/wiki/xacro">
+<robot name="all_sensors"
+  xmlns:xacro="http://www.ros.org/wiki/xacro">
   <!-- Imu -->
   <xacro:include filename="$(find rover_description)/urdf/sensors/imu.urdf.xacro" />

File: rover_description/urdf/sensors/asus_xtion.urdf.xacro (robot description, xacro)
@@ -21,8 +21,8 @@
     <xacro:property name="math_pi_over_2" value="1.5707963267948966" />
     <joint name="${prefix}_joint" type="fixed">
-        <axis xyz="1 0 0"/>
-        <xacro:insert_block name="origin"/>
-        <parent link="${parent}"/>
-        <child link="${prefix}_link"/>
+      <axis xyz="1 0 0"/>
+      <xacro:insert_block name="origin"/>
+      <parent link="${parent}"/>
+      <child link="${prefix}_link"/>
     </joint>
     <link name="${prefix}_link">
@@ -42,7 +42,5 @@
         <mass value="0.01" />
         <origin xyz="0 0 0" />
-        <inertia ixx="0.001" ixy="0.0" ixz="0.0"
-          iyy="0.001" iyz="0.0"
-          izz="0.001" />
+        <inertia ixx="0.001" ixy="0.0" ixz="0.0" iyy="0.001" iyz="0.0" izz="0.001" />
       </inertial>
     </link>
@@ -56,7 +54,5 @@
         <mass value="0.001" />
         <origin xyz="0 0 0" />
-        <inertia ixx="0.001" ixy="0.0" ixz="0.0"
-          iyy="0.001" iyz="0.0"
-          izz="0.001" />
+        <inertia ixx="0.001" ixy="0.0" ixz="0.0" iyy="0.001" iyz="0.0" izz="0.001" />
       </inertial>
     </link>

File: rover_description/urdf/sensors/hokuyo.urdf.xacro (robot description, xacro)
@@ -34,5 +34,5 @@
         <origin xyz="0 0 -0.05" rpy="0 0 0"/>
         <geometry>
-            <mesh filename="package://rover_description/meshes/sensors/hokuyo/hokuyo_ust_20lx.dae"/>
+          <mesh filename="package://rover_description/meshes/sensors/hokuyo/hokuyo_ust_20lx.dae"/>
         </geometry>
       </visual>
@@ -44,5 +44,5 @@
     </link>
     <gazebo reference="${prefix}_base_link">
-        <material>Gazebo/DarkGrey</material>
+      <material>Gazebo/DarkGrey</material>
     </gazebo>
     <link name="${prefix}_link">
@@ -54,33 +54,33 @@
     </joint>
     <gazebo reference="${prefix}_link">
-        <sensor name="lidar" type="gpu_lidar">"
-            <ignition_frame_id>${prefix}_link</ignition_frame_id>
-            <pose relative_to="${prefix}_link">0 0 0 0 0 0</pose>
-            <topic>/scan</topic>
-            <update_rate>10</update_rate>
-            <ray>
-                <scan>
-                    <horizontal>
-                        <samples>1081</samples>
-                        <resolution>1</resolution>
-                        <min_angle>${min_angle}</min_angle>
-                        <max_angle>${max_angle}</max_angle>
-                    </horizontal>
-                    <vertical>
-                        <samples>1</samples>
-                        <resolution>0.01</resolution>
-                        <min_angle>0</min_angle>
-                        <max_angle>0</max_angle>
-                    </vertical>
-                </scan>
-                <range>
-                    <min>0.06</min>
-                    <max>5.0</max>
-                    <resolution>0.01</resolution>
-                </range>
-            </ray>
-            <always_on>1</always_on>
-            <visualize>true</visualize>
-        </sensor>
+      <sensor name="lidar" type="gpu_lidar">"
+        <ignition_frame_id>${prefix}_link</ignition_frame_id>
+        <pose relative_to="${prefix}_link">0 0 0 0 0 0</pose>
+        <topic>/scan</topic>
+        <update_rate>10</update_rate>
+        <ray>
+          <scan>
+            <horizontal>
+              <samples>1081</samples>
+              <resolution>1</resolution>
+              <min_angle>${min_angle}</min_angle>
+              <max_angle>${max_angle}</max_angle>
+            </horizontal>
+            <vertical>
+              <samples>1</samples>
+              <resolution>0.01</resolution>
+              <min_angle>0</min_angle>
+              <max_angle>0</max_angle>
+            </vertical>
+          </scan>
+          <range>
+            <min>0.06</min>
+            <max>5.0</max>
+            <resolution>0.01</resolution>
+          </range>
+        </ray>
+        <always_on>1</always_on>
+        <visualize>true</visualize>
+      </sensor>
     </gazebo>
   </xacro:macro>

File: rover_description/urdf/sensors/imu.urdf.xacro (robot description, xacro)
@@ -20,8 +20,8 @@
   <xacro:macro name="sensor_imu" params="prefix parent *origin">
     <joint name="${prefix}_joint" type="fixed">
-        <axis xyz="1 0 0"/>
-        <xacro:insert_block name="origin"/>
-        <parent link="${parent}"/>
-        <child link="${prefix}_link"/>
+      <axis xyz="1 0 0"/>
+      <xacro:insert_block name="origin"/>
+      <parent link="${parent}"/>
+      <child link="${prefix}_link"/>
     </joint>
     <link name="${prefix}_link">
@@ -46,5 +46,5 @@
     </link>
     <gazebo reference="${prefix}_link">
-        <material>Gazebo/Blue</material>
+      <material>Gazebo/Blue</material>
     </gazebo>
     <gazebo reference="${prefix}_link">
