Commit message: Add factory_v2 world with lidar-fused SLAM
Convert factory_v2 from gz-sim to Gazebo Classic: drop the gz::sim system
plugins, point the cardboard box mesh and the door materials at local assets
instead of Fuel, and remove the <state> snapshot so Classic reads model poses
directly.

RTAB-Map hardcoded subscribe_scan to False and Grid/Sensor to 1, so the hokuyo
published /scan that nothing consumed. Expose subscribe_scan as a launch
argument that also switches Grid/Sensor between depth-only and depth+lidar, and
default it to True for this world.

The simulated depth camera only manages a few frames per second, so odom_rgbd
loses tracking as soon as the rover moves and stalls the EKF. Split the sim
config into ekf_sim.yaml, which fuses wheel_odom, and select it from
use_sim_time; hardware still fuses odom_rgbd through the unchanged ekf.yaml.

Pitch the RGB-D camera up so it sees shelving and walls rather than floor, and
document cloning this fork's humble branch, since the fork defaults to jazzy.

Co-Authored-By: Claude Opus 5 (1M context) <noreply@anthropic.com>

File: rover_description/robots/rover.urdf.xacro (robot description, xacro)
@@ -185,5 +185,6 @@
     </xacro:sensor_imu>
     <xacro:sensor_asus_xtion prefix="camera" parent="base_link">
-        <origin xyz="0.215 0 0.065" rpy="0 0.4 0"/>
+        <!-- negative pitch tilts the RGB-D camera up, towards shelving and walls -->
+        <origin xyz="0.215 0 0.065" rpy="0 -0.2 0"/>
         <!-- <origin xyz="0.212 0 0.065" rpy="0 0 0"/> -->
     </xacro:sensor_asus_xtion>
